File: Hardware/feather-candle/feather-candle.sch (KiCad schematic (older format))
At the start: 22 parts, among them J1 CONN_05, J2 CONN_05, J3 CONN_05, J4 CONN_121X12_NO_SILK_KIT, J5 CONN_121X12_NO_SILK_KIT, J6 CONN_161X16_NO_SILK, J7 CONN_161X16_NO_SILK

Commit message: Fixed several issues with the PCB layout. Correct hole placement of the 1042 battery holder. Correct mounting hole placement of the Feather boards. Changed resistor footprints to 1206 and 0805_HandSoldering. Deleted the keepout-area around the heart shape.
Parts:
- BT1: footprint SparkfunBatteries:BATTERY_18650-HOLDER_1024P -> Keystone_BatteryHolder:BATTERY_18650-HOLDER_1042P
- C1, C2: footprint Capacitors_SMD:C_0805 -> Capacitors_SMD:C_0805_HandSoldering
- C3, C4: footprint Capacitors_SMD:C_1210 -> Capacitors_SMD:C_1210_HandSoldering
- R1, R3, R4: footprint Resistors:0805 -> Resistors:1206
Changed lines of the file:
@@
 F 0 "BT1" V 2000 5900 45  0000 L BNN
 F 1 "BATTERY-18650" V 1650 5600 45  0000 L BNN
-F 2 "SparkfunBatteries:BATTERY_18650-HOLDER_1024P" H 1800 6500 20  0001 C CNN
+F 2 "Keystone_BatteryHolder:BATTERY_18650-HOLDER_1042P" H 1800 6500 20  0001 C CNN
 F 3 "" H 1800 6250 60  0001 C CNN
 F 4 "BATT-12327" H 1800 6550 60  0001 C CNN "Feld4"
@@
 F 0 "R1" H 8300 4300 45  0000 L BNN
 F 1 "10k" H 8300 4100 45  0000 L BNN
-F 2 "Resistors:0805" H 8500 4400 20  0001 C CNN
+F 2 "Resistors:1206" H 8500 4400 20  0001 C CNN
 F 3 "" H 8500 4250 60  0001 C CNN
 F 4 " " H 8500 4450 60  0000 C CNN "Feld4"
@@
 F 0 "C1" H 5375 2550 50  0000 L CNN
 F 1 "C" H 5375 2350 50  0000 L CNN
-F 2 "Capacitors_SMD:C_0805" H 5388 2300 50  0001 C CNN
+F 2 "Capacitors_SMD:C_0805_HandSoldering" H 5388 2300 50  0001 C CNN
 F 3 "" H 5350 2450 50  0001 C CNN
 	1    5350 2450
@@
 F 0 "C2" H 5625 2550 50  0000 L CNN
 F 1 "C" H 5625 2350 50  0000 L CNN
-F 2 "Capacitors_SMD:C_0805" H 5638 2300 50  0001 C CNN
+F 2 "Capacitors_SMD:C_0805_HandSoldering" H 5638 2300 50  0001 C CNN
 F 3 "" H 5600 2450 50  0001 C CNN
 	1    5600 2450
@@
 F 0 "C3" H 5875 2550 50  0000 L CNN
 F 1 "C" H 5875 2350 50  0000 L CNN
-F 2 "Capacitors_SMD:C_1210" H 5888 2300 50  0001 C CNN
+F 2 "Capacitors_SMD:C_1210_HandSoldering" H 5888 2300 50  0001 C CNN
 F 3 "" H 5850 2450 50  0001 C CNN
 	1    5850 2450
@@
 F 0 "C4" H 6125 2550 50  0000 L CNN
 F 1 "C" H 6125 2350 50  0000 L CNN
-F 2 "Capacitors_SMD:C_1210" H 6138 2300 50  0001 C CNN
+F 2 "Capacitors_SMD:C_1210_HandSoldering" H 6138 2300 50  0001 C CNN
 F 3 "" H 6100 2450 50  0001 C CNN
 	1    6100 2450
@@
 F 0 "R3" H 1250 5500 45  0000 L BNN
 F 1 "10k" H 1250 5300 45  0000 L BNN
-F 2 "Resistors:0805" H 1450 5600 20  0001 C CNN
+F 2 "Resistors:1206" H 1450 5600 20  0001 C CNN
 F 3 "" H 1450 5450 60  0001 C CNN
 F 4 " " H 1450 5650 60  0000 C CNN "Feld4"
@@
 F 0 "R4" H 4600 5650 45  0000 L BNN
 F 1 "10k" H 4600 5450 45  0000 L BNN
-F 2 "Resistors:0805" H 4800 5750 20  0001 C CNN
+F 2 "Resistors:1206" H 4800 5750 20  0001 C CNN
 F 3 "" H 4800 5600 60  0001 C CNN
 F 4 " " H 4800 5800 60  0000 C CNN "Feld4"
