File: Hardware/feather-candle/feather-candle.kicad_pcb (KiCad board)
At the start: 2 copper layers, 254 x 22.9 mm, 37 parts, among them J1 CONN_05, J2 CONN_05, J3 CONN_05, J4 CONN_121X12_NO_SILK_KIT, J5 CONN_121X12_NO_SILK_KIT, J6 CONN_161X16_NO_SILK, J7 CONN_161X16_NO_SILK

Commit message: first release
Routing:
- net +5V: track 249.3 -> 251.9 mm
- net /SDA_HUZZAH: track 180.4 -> 181.5 mm
- net /SCL_HUZZAH: track 179.0 -> 178.0 mm
Other:
- board text added: "github.com/mnemocron simonmartin.ch"
- board text removed: "github.com/mnemocron - simonmartin.ch"
